Commit message: fixed bugs; added world file; controller number error in cpp files; urdf bugs; inertia and gazebo files; error in namespaces, etc.

File: dlr_description/urdf/hit2/hit2.gazebo.xacro (robot description, xacro)
@@ -293,4 +293,9 @@
             </plugin>
         </gazebo>
+        <!-- <gazebo>
+          <plugin name="gazebo_ros_control" filename="libgazebo_ros_control.so">
+            <robotNamespace>${name}</robotNamespace>
+          </plugin>
+        </gazebo> -->
     </xacro:macro>
 </robot>

File: dlr_description/urdf/hit2/hit2.urdf (robot description, URDF)
Before this commit: robot lwr, 22 links, 21 joints
Links:
- link right_index_distal_link: geometry collision mesh filename=package://dlr_description/meshes/hit2/distal.stl; visual mesh filename=package://dlr_description/meshes/hit2/distal.stl
- link right_index_medial_link: geometry collision mesh filename=package://dlr_description/meshes/hit2/medial.stl; visual mesh filename=package://dlr_description/meshes/hit2/medial.stl
- link right_index_proximal_link: geometry collision mesh filename=package://dlr_description/meshes/hit2/proximal.stl; visual mesh filename=package://dlr_description/meshes/hit2/proximal.stl
- link right_middle_distal_link: geometry collision mesh filename=package://dlr_description/meshes/hit2/distal.stl; visual mesh filename=package://dlr_description/meshes/hit2/distal.stl
- link right_middle_medial_link: geometry collision mesh filename=package://dlr_description/meshes/hit2/medial.stl; visual mesh filename=package://dlr_description/meshes/hit2/medial.stl
- link right_middle_proximal_link: geometry collision mesh filename=package://dlr_description/meshes/hit2/proximal.stl; visual mesh filename=package://dlr_description/meshes/hit2/proximal.stl
- link right_pinky_distal_link: geometry collision mesh filename=package://dlr_description/meshes/hit2/distal.stl; visual mesh filename=package://dlr_description/meshes/hit2/distal.stl
- link right_pinky_medial_link: geometry collision mesh filename=package://dlr_description/meshes/hit2/medial.stl; visual mesh filename=package://dlr_description/meshes/hit2/medial.stl
- link right_pinky_proximal_link: geometry collision mesh filename=package://dlr_description/meshes/hit2/proximal.stl; visual mesh filename=package://dlr_description/meshes/hit2/proximal.stl
- link right_ring_distal_link: geometry collision mesh filename=package://dlr_description/meshes/hit2/distal.stl; visual mesh filename=package://dlr_description/meshes/hit2/distal.stl
- link right_ring_medial_link: geometry collision mesh filename=package://dlr_description/meshes/hit2/medial.stl; visual mesh filename=package://dlr_description/meshes/hit2/medial.stl
- link right_ring_proximal_link: geometry collision mesh filename=package://dlr_description/meshes/hit2/proximal.stl; visual mesh filename=package://dlr_description/meshes/hit2/proximal.stl
- link right_thumb_distal_link: geometry collision mesh filename=package://dlr_description/meshes/hit2/distal.stl; visual mesh filename=package://dlr_description/meshes/hit2/distal.stl
- link right_thumb_medial_link: geometry collision mesh filename=package://dlr_description/meshes/hit2/medial.stl; visual mesh filename=package://dlr_description/meshes/hit2/medial.stl
- link right_thumb_proximal_link: geometry collision mesh filename=package://dlr_description/meshes/hit2/proximal.stl; visual mesh filename=package://dlr_description/meshes/hit2/proximal.stl
